File: RGBStripe_FFT/schematic/rgbstripe_fft_pcb.brd (EAGLE design)
At the start: 46.9 x 61.5 mm, 21 parts, among them IC1 MSGEQ7P, J1 POWER_JACK, M1 ARDUINO-NANO-3.0

Commit message: added Sketch + Schematic using FFT instead of MSGEQ7 Circuit
Parts:
- removed 100NF, C4: 33pF, resistor:C025-025X050
- removed 100NF1: 10nF, resistor:C025-025X050
- removed AUX: (no value), con-lstb:MA03-1
- removed BRIGHT_SLIDER: PC16S, piher:PC16S
- removed C2: 100nF, resistor:C025-025X050
- removed IC1: MSGEQ7P, SparkFun-IC-Special-Function:DIP08
- removed MSGEQ7-FEMALE, MSGEQ7-MALE: (no value), con-lstb:MA05-1
- removed PWR: (no value), pinhead:1X02
- removed R1: 200k, resistor:0204/5
- removed S1: MODE_SWITCH, SparkFun-Switches:TACTILE_SWITCH_PTH_12MM
- added J2: AUDIO_JACK_3.5MM_KIT, SparkFun-Connectors:AUDIO-JACK-KIT
- added R4: (no value), pot:3RP/1610N
- added SW: 22-23-2021, con-molex:22-23-2021
- M1: device diy-modules:ARDUINO-NANO-3.0 -> diy-modules-nano:ARDUINO-NANO-3.0
- moved J1 251.9 mm to (147.3, 104.1), turned to 180 degrees
- moved R2 202.3 mm to (134.6, 87.6), turned to 270 degrees
- moved C3 193.6 mm to (141.0, 85.1), turned to 180 degrees
- moved WS2812 190.8 mm to (134.6, 94.0)
- moved C1 167.3 mm to (126.9, 72.4), turned to 180 degrees
- moved R3 151.9 mm to (126.2, 54.6), turned to 90 degrees
- moved D1 120.9 mm to (123.2, 74.9), turned to 180 degrees
- moved M1 114.8 mm to (138.4, 69.8)
- moved PWR-SWITCH 111.8 mm to (156.2, 85.1), turned to 270 degrees
Connections:
- removed net GNDA: BRIGHT_SLIDER.1E, C3.1, C4.1, J1.PWR, M1.J1.4, M1.J2.2, MSGEQ7-FEMALE.3, PWR.1, R3.2, WS2812.3
- removed net N$10: 100NF1.1, AUX.1, AUX.2
- removed net N$11: C4.2, IC1.8, R1.1
- removed net N$12: 100NF.1, AUX.3, IC1.2
- removed net N$13: 100NF1.2, IC1.5
- removed net N$2: M1.J1.8, MSGEQ7-FEMALE.5
- removed net N$3: M1.J2.11, MSGEQ7-FEMALE.2
- removed net N$4: M1.J1.5, MSGEQ7-FEMALE.1
- removed net N$5: C2.2, IC1.1, MSGEQ7-MALE.2
- removed net N$7: IC1.3, MSGEQ7-MALE.4
- removed net N$9: IC1.7, MSGEQ7-MALE.1
- new net GND: C1.2, C3.1, J1.GND, J1.GNDBREAK, J2.SLEEVE, M1.J1.4, M1.J2.2, R3.2, R4.3, WS2812.3
- new net N$19: J1.PWR, PWR-SWITCH.2
- net N$1: now also C1.1
- net N$15: now also R4.2; no longer BRIGHT_SLIDER.1S
- net N$17: now also SW.1; no longer S1.3
- net N$6: now also J2.RING, M1.J2.11; no longer 100NF.2, C2.1, IC1.6, MSGEQ7-MALE.3
- net N$8: now also M1.J1.5; no longer IC1.4, MSGEQ7-MALE.5
- net VCC: now also R4.1, SW.2; no longer BRIGHT_SLIDER.1A, C1.1, C1.2, J1.GND, J1.GNDBREAK, MSGEQ7-FEMALE.4, PWR-SWITCH.2, PWR.2, R1.2, S1.1
Routing:
- added copper zone on layer 16, net GND
Other:
- board size 46.9 x 61.5 mm -> 46 x 52.1 mm
