File: RGB_Backlight_FFT_Test/schematic/rgbstripe_fft_lochraster.brd (EAGLE design)
At the start: 46 x 62.3 mm, 15 parts, among them J1 POWER_JACK, J2 AUDIO_JACK_3.5MM_KIT, M1 ARDUINO-NANO-3.0

Commit message: case: 123Design case added + Sketches Updates
Parts:
- C1: device resistor:C025-025X050 -> resistor:C050-024X044
- R3: value 10k -> 220k
- moved C1 1.27 mm to (125.6, 67.3)
Connections:
- net N$1: now also R4.1, SW.2
- net VCC: no longer R4.1, SW.2
Routing:
- net VCC: track 125.4 -> 56.8 mm
- net N$1: track 5.21 -> 67.2 mm, vias 0 -> 1
Changed lines of the file:
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@@
 </autorouter>
 <elements>
-<element name="C1" library="resistor" library_urn="urn:adsk.eagle:library:348" package="C025-025X050" package3d_urn="urn:adsk.eagle:package:26151/1" value="10nF" x="126.873" y="67.31" smashed="yes" rot="R180">
-<attribute name="NAME" x="129.159" y="65.786" size="1.27" layer="25" ratio="10" rot="R180"/>
-<attribute name="VALUE" x="129.159" y="70.104" size="1.27" layer="27" ratio="10" rot="R180"/>
+<element name="C1" library="resistor" library_urn="urn:adsk.eagle:library:348" package="C050-024X044" package3d_urn="urn:adsk.eagle:package:26162/1" value="10nF" x="125.603" y="67.31" smashed="yes" rot="R180">
+<attribute name="NAME" x="127.889" y="65.786" size="1.27" layer="25" ratio="10" rot="R180"/>
+<attribute name="VALUE" x="127.889" y="70.104" size="1.27" layer="27" ratio="10" rot="R180"/>
 </element>
 <element name="C3" library="resistor" library_urn="urn:adsk.eagle:library:348" package="E3,5-8" package3d_urn="urn:adsk.eagle:package:25842/1" value="1000uF" x="140.97" y="82.55" smashed="yes" rot="R180">
@@
 <attribute name="VALUE" x="131.6736" y="89.9414" size="0.9906" layer="27" ratio="10" rot="R180"/>
 </element>
-<element name="R3" library="resistor" library_urn="urn:adsk.eagle:library:348" package="0204/7" package3d_urn="urn:adsk.eagle:package:25945/1" value="10k" x="126.238" y="48.26" smashed="yes" rot="R90">
+<element name="R3" library="resistor" library_urn="urn:adsk.eagle:library:348" package="0204/7" package3d_urn="urn:adsk.eagle:package:25945/1" value="220k" x="126.238" y="48.26" smashed="yes" rot="R90">
 <attribute name="NAME" x="125.0696" y="46.2534" size="0.9906" layer="25" ratio="10" rot="R90"/>
 <attribute name="VALUE" x="128.5494" y="46.1264" size="0.9906" layer="27" ratio="10" rot="R90"/>
@@
 <contactref element="PWR-SWITCH" pad="3"/>
 <contactref element="D1" pad="A"/>
-<contactref element="SW" pad="2"/>
-<contactref element="R4" pad="1"/>
-<wire x1="138.51" y1="41.783" x2="130.81" y2="41.783" width="2" layer="16"/>
-<wire x1="130.81" y1="44.45" x2="130.81" y2="41.783" width="2" layer="16"/>
 <wire x1="139.192" y1="82.55" x2="138.43" y2="80.01" width="2" layer="16"/>
 <wire x1="138.43" y1="80.01" x2="130.81" y2="80.01" width="2" layer="16"/>
@@
 <wire x1="139.192" y1="82.55" x2="133.35" y2="82.55" width="2" layer="16"/>
 <wire x1="133.35" y1="82.55" x2="133.35" y2="92.71" width="2" layer="16"/>
-<wire x1="118.11" y1="69.85" x2="118.11" y2="49.53" width="2" layer="16"/>
-<wire x1="118.11" y1="49.53" x2="123.19" y2="49.53" width="2" layer="16"/>
-<wire x1="130.81" y1="41.783" x2="123.19" y2="41.783" width="2" layer="16"/>
-<wire x1="123.19" y1="41.783" x2="123.19" y2="49.53" width="2" layer="16"/>
 <wire x1="118.11" y1="69.85" x2="118.11" y2="80.01" width="2" layer="16"/>
-<wire x1="158.5268" y1="63.9412" x2="138.51" y2="41.783" width="0" layer="19" extent="16-16"/>
-<wire x1="154.94" y1="80.01" x2="154.94" y2="80.01" width="2" layer="16"/>
-<wire x1="157.6752" y1="76.0649375" x2="157.6752" y2="64.7928" width="0.9144" layer="16"/>
-<wire x1="157.6752" y1="64.7928" x2="158.5268" y2="63.9412" width="0.9144" layer="16"/>
-<wire x1="154.94" y1="80.01" x2="154.94" y2="78.8001375" width="0.9144" layer="16"/>
-<wire x1="154.94" y1="78.8001375" x2="157.6752" y2="76.0649375" width="0.9144" layer="16"/>
+<wire x1="118.11" y1="80.01" x2="130.81" y2="80.01" width="0" layer="19" extent="16-16"/>
 </signal>
 <signal name="N$1">
@@
 <wire x1="128.27" y1="72.39" x2="128.27" y2="69.85" width="2" layer="16"/>
 <wire x1="128.27" y1="69.85" x2="128.27" y2="67.31" width="2" layer="16"/>
-<wire x1="128.27" y1="67.31" x2="128.143" y2="67.31" width="2" layer="16"/>
+<contactref element="SW" pad="2"/>
+<contactref element="R4" pad="1"/>
+<wire x1="138.51" y1="41.783" x2="138.51" y2="44.45" width="2" layer="16"/>
+<wire x1="138.51" y1="44.45" x2="130.81" y2="44.45" width="2" layer="16"/>
+<wire x1="130.81" y1="44.45" x2="130.524" y2="44.45" width="2" layer="16"/>
+<wire x1="130.524" y1="44.45" x2="130.524" y2="41.4848" width="2" layer="16"/>
+<wire x1="130.524" y1="41.4848" x2="123.19" y2="41.4848" width="2" layer="16"/>
+<wire x1="123.19" y1="41.4848" x2="123.19" y2="46.99" width="2" layer="16"/>
+<wire x1="123.19" y1="46.99" x2="118.11" y2="46.99" width="2" layer="16"/>
+<wire x1="118.11" y1="46.99" x2="118.11" y2="64.77" width="2" layer="16"/>
+<via x="118.11" y="64.77" extent="1-16" drill="1"/>
+<wire x1="118.11" y1="64.77" x2="128.27" y2="64.77" width="2" layer="1"/>
+<wire x1="128.143" y1="67.31" x2="128.27" y2="67.31" width="2" layer="16"/>
+<wire x1="128.27" y1="67.31" x2="128.27" y2="64.77" width="2" layer="16"/>
+<wire x1="128.27" y1="64.77" x2="128.27" y2="64.77" width="0" layer="19" extent="1-16"/>
 </signal>
 <signal name="N$8">
@@
 <wire x1="138.43" y1="92.71" x2="138.43" y2="97.79" width="2" layer="16"/>
 <wire x1="138.43" y1="97.79" x2="123.19" y2="97.79" width="2" layer="16"/>
-<wire x1="123.19" y1="67.31" x2="125.603" y2="67.31" width="2" layer="16"/>
+<wire x1="123.19" y1="67.31" x2="123.063" y2="67.31" width="2" layer="16"/>
 <wire x1="123.19" y1="67.31" x2="123.19" y2="72.39" width="2" layer="16"/>
-<wire x1="128.27" y1="62.23" x2="125.73" y2="62.23" width="2" layer="16"/>
-<wire x1="125.73" y1="62.23" x2="125.73" y2="67.31" width="2" layer="16"/>
-<wire x1="125.603" y1="67.31" x2="125.73" y2="67.31" width="2" layer="16"/>
 <wire x1="148.51" y1="41.783" x2="148.51" y2="49.53" width="2" layer="16"/>
 <wire x1="128.27" y1="62.23" x2="128.27" y2="57.15" width="2" layer="16"/>
@@
 <wire x1="138.43" y1="92.71" x2="138.43" y2="87.63" width="2" layer="16"/>
 <wire x1="138.43" y1="87.63" x2="142.748" y2="87.63" width="2" layer="16"/>
+<wire x1="123.063" y1="67.31" x2="123.063" y2="62.23" width="2" layer="16"/>
+<wire x1="123.063" y1="62.23" x2="128.27" y2="62.23" width="2" layer="16"/>
 </signal>
 <signal name="N$19">
@@
 <wire x1="128.29" y1="85.09" x2="128.27" y2="85.09" width="2" layer="16"/>
 </signal>
+<signal name="N$4">
+<via x="128.27" y="64.77" extent="1-16" drill="1"/>
+</signal>
 </signals>
