File: RGB_Backlight_FFT/schematic/rgbstripe_fft_lochraster.brd (EAGLE design)
At the start: 46 x 62.3 mm, 15 parts, among them J1 POWER_JACK, J2 AUDIO_JACK_3.5MM_KIT, M1 ARDUINO-NANO-3.0

Commit message: finished 3D print case
Parts:
- moved R4 7.62 mm to (151.1, 41.8)
Routing:
- net N$1: track 67.2 -> 74.8 mm
- net GND: track 161.8 -> 154.2 mm
Changed lines of the file:
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@@
 <attribute name="VALUE" x="127" y="39.37" size="1.016" layer="27" ratio="10"/>
 </element>
-<element name="R4" library="pot" library_urn="urn:adsk.eagle:library:331" package="3RP/1610N" package3d_urn="urn:adsk.eagle:package:22726/1" value="" x="143.51" y="41.783" smashed="yes">
-<attribute name="NAME" x="135.255" y="47.498" size="1.27" layer="25"/>
-<attribute name="POPULARITY" value="8" x="143.51" y="41.783" size="1.778" layer="27" display="off"/>
-<attribute name="VALUE" x="140.335" y="44.323" size="1.27" layer="27"/>
+<element name="R4" library="pot" library_urn="urn:adsk.eagle:library:331" package="3RP/1610N" package3d_urn="urn:adsk.eagle:package:22726/1" value="" x="151.13" y="41.783" smashed="yes">
+<attribute name="NAME" x="142.875" y="47.498" size="1.27" layer="25"/>
+<attribute name="POPULARITY" value="8" x="151.13" y="41.783" size="1.778" layer="27" display="off"/>
+<attribute name="VALUE" x="147.955" y="44.323" size="1.27" layer="27"/>
 </element>
 <element name="SV1" library="con-lsta" library_urn="urn:adsk.eagle:library:161" package="FE15" package3d_urn="urn:adsk.eagle:package:8206/1" value="" x="138.43" y="54.61" smashed="yes" rot="R180">
@@
 <contactref element="SW" pad="2"/>
 <contactref element="R4" pad="1"/>
-<wire x1="138.51" y1="41.783" x2="138.51" y2="44.45" width="2" layer="16"/>
-<wire x1="138.51" y1="44.45" x2="130.81" y2="44.45" width="2" layer="16"/>
+<wire x1="146.13" y1="41.783" x2="146.13" y2="44.45" width="2" layer="16"/>
+<wire x1="146.13" y1="44.45" x2="130.81" y2="44.45" width="2" layer="16"/>
 <wire x1="130.81" y1="44.45" x2="130.524" y2="44.45" width="2" layer="16"/>
 <wire x1="130.524" y1="44.45" x2="130.524" y2="41.4848" width="2" layer="16"/>
@@
 <contactref element="M1" pad="J2.10"/>
 <contactref element="R4" pad="2"/>
-<wire x1="143.51" y1="41.783" x2="143.51" y2="72.39" width="0" layer="19" extent="1-1"/>
+<wire x1="151.13" y1="41.783" x2="143.51" y2="72.39" width="0" layer="19" extent="1-1"/>
 </signal>
 <signal name="GND">
@@
 <wire x1="123.19" y1="67.31" x2="123.063" y2="67.31" width="2" layer="16"/>
 <wire x1="123.19" y1="67.31" x2="123.19" y2="72.39" width="2" layer="16"/>
-<wire x1="148.51" y1="41.783" x2="148.51" y2="49.53" width="2" layer="16"/>
+<wire x1="156.13" y1="41.783" x2="156.13" y2="49.53" width="2" layer="16"/>
 <wire x1="128.27" y1="62.23" x2="128.27" y2="57.15" width="2" layer="16"/>
 <wire x1="128.27" y1="57.15" x2="128.27" y2="52.07" width="2" layer="16"/>
 <wire x1="126.238" y1="52.07" x2="128.27" y2="52.07" width="2" layer="16"/>
-<wire x1="148.51" y1="49.53" x2="158.75" y2="49.53" width="2" layer="16"/>
+<wire x1="156.13" y1="49.53" x2="158.75" y2="49.53" width="2" layer="16"/>
 <wire x1="158.75" y1="49.53" x2="158.75" y2="62.23" width="2" layer="16"/>
 <wire x1="158.75" y1="62.23" x2="128.27" y2="62.23" width="2" layer="16"/>
